File: MerlinGame.kicad_pcb (KiCad board)
At the start: 2 copper layers, 60 x 125 mm, 39 parts, among them J1 AVR-ISP-6, J2 BATTERY, SW1 0, SW10 9, SW11 10, SW12 NEW GAME, SW13 SAME GAME, SW14 HIT ME, SW15 COMP TURN, SW16 POWER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

Commit message: Routing
Parts:
- RN1, RN2, RN3: value 1K -> 330
- moved J1 2.31 mm to (61.0, 152.0), turned to 0 degrees
- moved C1 1.00 mm to (88.0, 153.0)
- moved C2 1.00 mm to (88.0, 151.0)
- moved C3 1.00 mm to (88.0, 157.0)
- moved C4 1.00 mm to (70.0, 155.0)
- moved C5 1.00 mm to (70.0, 153.0)
- moved C6 1.00 mm to (88.0, 155.0)
- moved R1 1.00 mm to (70.0, 151.0)
- moved R2 1.00 mm to (70.0, 157.0)
- moved R3 1.00 mm to (70.0, 159.0)
- moved Y1 1.00 mm to (96.0, 158.0)
Routing:
- net GND: track 0.00 -> 500.9 mm, vias 0 -> 12
- net VCC: track 0.00 -> 202.3 mm, vias 0 -> 5
- net /K4: track 0.00 -> 197.9 mm, vias 0 -> 2
- net /O0: track 0.00 -> 180.3 mm, vias 0 -> 1
- net /K8: track 0.00 -> 157.9 mm, vias 0 -> 1
- net /K1: track 0.00 -> 156.8 mm, vias 0 -> 1
- net /K2: track 0.00 -> 155.8 mm
- net /O1: track 0.00 -> 137.0 mm, vias 0 -> 1
- net /BUZZER: track 0.00 -> 121.1 mm, vias 0 -> 1
- net /O2: track 0.00 -> 108.5 mm, vias 0 -> 1
- net /LED0: track 0.00 -> 101.5 mm, vias 0 -> 1
- net /LED3: track 0.00 -> 98.2 mm, vias 0 -> 1
- net /LED1: track 0.00 -> 90.7 mm, vias 0 -> 1
- net /LED6: track 0.00 -> 86.5 mm, vias 0 -> 1
- net /LED2: track 0.00 -> 81.5 mm, vias 0 -> 1
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- added copper zone on B.Cu, net GND
- added copper zone on F.Cu, net GND
Other:
- net class Default: clearance 0.2 -> 0.15; trace_width 0.25 -> 0.15; via_dia 0.8 -> 0.6; via_drill 0.4 -> 0.3
- net class POWER added: clearance 0.2, trace_width 0.3, via_dia 0.8, via_drill 0.4
- net class VBATT added: clearance 0.2, trace_width 0.5, via_dia 0.8, via_drill 0.4
- rule pad_to_mask_clearance: 0.2 -> 0.1
- rule trace_clearance: 0.2 -> 0.15
- rule trace_min: 0.2 -> 0.15
- rule via_min_size: 0.4 -> 0.6

Commit message: Updated silkscreen, added plots
Parts:
- C1, C2: value 22pF -> 18pF
Other:
- board text added: "JLCJLCJLCJLC"
- board text added: "Wizard Game Rev A 2019 Dominic Thibodeau dev@hotkeysoft.net"
Changed lines of the file:
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@@
   (general
     (thickness 1.6)
-    (drawings 20)
+    (drawings 22)
     (tracks 616)
     (zones 0)
@@
     (35 F.Paste user)
     (36 B.SilkS user)
-    (37 F.SilkS user)
+    (37 F.SilkS user hide)
     (38 B.Mask user)
     (39 F.Mask user)
@@
     (47 F.CrtYd user)
     (48 B.Fab user hide)
-    (49 F.Fab user hide)
+    (49 F.Fab user)
   )
   (setup
@@
     (visible_elements 7FFFFFFF)
     (pcbplotparams
-      (layerselection 0x010fc_ffffffff)
+      (layerselection 0x010f0_ffffffff)
       (usegerberextensions false)
       (usegerberattributes false)
@@
       (outputformat 1)
       (mirror false)
-      (drillshape 1)
+      (drillshape 0)
       (scaleselection 1)
-      (outputdirectory ""))
+      (outputdirectory "plot"))
   )
   (net 0 "")
@@
       (effects (font (size 1 1) (thickness 0.15)) (justify mirror))
     )
-    (fp_text value SPEAKER (at 3 -1 90) (layer B.SilkS)
+    (fp_text value SPEAKER (at -0.135 -5.08 180) (layer B.SilkS)
       (effects (font (size 1 1) (thickness 0.15)) (justify mirror))
     )
@@
       (effects (font (size 1 1) (thickness 0.15)) (justify mirror))
     )
-    (fp_text value BATTERY (at 3 -1 -90) (layer B.SilkS)
+    (fp_text value BATTERY (at 0 -5.08 180) (layer B.SilkS)
       (effects (font (size 1 1) (thickness 0.15)) (justify mirror))
     )
@@
       (effects (font (size 1 1) (thickness 0.15)))
     )
-    (fp_text value 22pF (at 0 2 180) (layer F.Fab)
+    (fp_text value 18pF (at 0 2 180) (layer F.Fab)
       (effects (font (size 1 1) (thickness 0.15)))
     )
@@
       (effects (font (size 1 1) (thickness 0.15)))
     )
-    (fp_text value 22pF (at 0 1.65 180) (layer F.Fab)
+    (fp_text value 18pF (at 0 1.65 180) (layer F.Fab)
       (effects (font (size 1 1) (thickness 0.15)))
     )
@@
     )
   )
-  (gr_text SPEAKER (at 66.04 52.197 90) (layer F.SilkS)
+  (gr_text JLCJLCJLCJLC (at 80 163.068) (layer B.SilkS)
+    (effects (font (size 1 1) (thickness 0.15)) (justify mirror))
+  )
+  (gr_text "Wizard Game Rev A\n2019 Dominic Thibodeau\ndev@hotkeysoft.net" (at 103.505 58.42) (layer B.SilkS)
+    (effects (font (size 1 1) (thickness 0.15)) (justify left mirror))
+  )
+  (gr_text SPEAKER (at 62.865 55.5) (layer F.SilkS)
     (effects (font (size 1 1) (thickness 0.15)))
   )
-  (gr_text BATTERY (at 98.298 52.324 90) (layer F.SilkS)
+  (gr_text BATTERY (at 95.25 55.5) (layer F.SilkS)
     (effects (font (size 1 1) (thickness 0.15)))
   )

Commit message: Removed battery holes
Parts:
- removed MH5: BATTERY1, MountingHole:MountingHole_2.7mm_Pad
- removed MH6: BATTERY2, MountingHole:MountingHole_2.7mm_Pad
Routing:
- net GND: track 500.9 -> 489.1 mm, vias 12 -> 13
- net /LED7: track 44.1 -> 43.1 mm
Other:
- board text removed: "+"
- board text removed: "-"
Changed lines of the file:
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@@
   (general
     (thickness 1.6)
-    (drawings 22)
-    (tracks 616)
+    (drawings 14)
+    (tracks 618)
     (zones 0)
-    (modules 39)
+    (modules 37)
     (nets 44)
   )
@@
     (35 F.Paste user)
     (36 B.SilkS user)
-    (37 F.SilkS user hide)
+    (37 F.SilkS user)
     (38 B.Mask user)
     (39 F.Mask user)
@@
   )
   (module MountingHole:MountingHole_2.7mm_Pad (layer F.Cu)
-    (at 69 135)
-    (descr "Mounting Hole 2.7mm")
-    (tags "mounting hole 2.7mm")
-    (attr virtual)
-    (fp_text reference MH5 (at 0 -3.7) (layer F.SilkS) hide
-      (effects (font (size 1 1) (thickness 0.15)))
-    )
-    (fp_text value BATTERY1 (at 0 3.7) (layer F.Fab)
-      (effects (font (size 1 1) (thickness 0.15)))
-    )
-    (fp_circle (center 0 0) (end 2.95 0) (layer F.CrtYd) (width 0.05))
-    (fp_circle (center 0 0) (end 2.7 0) (layer Cmts.User) (width 0.15))
-    (fp_text user %R (at 0.3 0) (layer F.Fab)
-      (effects (font (size 1 1) (thickness 0.15)))
-    )
-    (pad 1 thru_hole circle (at 0 0) (size 5.4 5.4) (drill 2.7) (layers *.Cu *.Mask)
-      (net 3 GND))
-  )
-  (module MountingHole:MountingHole_2.7mm_Pad (layer F.Cu)
     (at 105 160)
     (descr "Mounting Hole 2.7mm")
@@
     )
     (fp_text value CASE (at 0 3.7) (layer F.Fab)
-      (effects (font (size 1 1) (thickness 0.15)))
-    )
-    (fp_circle (center 0 0) (end 2.95 0) (layer F.CrtYd) (width 0.05))
-    (fp_circle (center 0 0) (end 2.7 0) (layer Cmts.User) (width 0.15))
-    (fp_text user %R (at 0.3 0) (layer F.Fab)
-      (effects (font (size 1 1) (thickness 0.15)))
-    )
-    (pad 1 thru_hole circle (at 0 0) (size 5.4 5.4) (drill 2.7) (layers *.Cu *.Mask)
-      (net 3 GND))
-  )
-  (module MountingHole:MountingHole_2.7mm_Pad (layer F.Cu)
-    (at 91 135)
-    (descr "Mounting Hole 2.7mm")
-    (tags "mounting hole 2.7mm")
-    (attr virtual)
-    (fp_text reference MH6 (at 0 -3.7) (layer F.SilkS) hide
-      (effects (font (size 1 1) (thickness 0.15)))
-    )
-    (fp_text value BATTERY2 (at 0 3.7) (layer F.Fab)
       (effects (font (size 1 1) (thickness 0.15)))
     )
@@
     (effects (font (size 1 1) (thickness 0.15)))
   )
-  (gr_text - (at 60.325 53.467 180) (layer F.SilkS)
-    (effects (font (size 1.5 1.5) (thickness 0.3)))
-  )
-  (gr_text + (at 60.325 50.927 180) (layer F.SilkS)
-    (effects (font (size 1.5 1.5) (thickness 0.3)))
-  )
-  (gr_text + (at 92.075 50.927 180) (layer F.SilkS)
-    (effects (font (size 1.5 1.5) (thickness 0.3)))
-  )
-  (gr_text - (at 92.075 53.467 180) (layer F.SilkS)
-    (effects (font (size 1.5 1.5) (thickness 0.3)))
-  )
-  (gr_text - (at 92.075 53.213) (layer B.SilkS)
-    (effects (font (size 1.5 1.5) (thickness 0.3)) (justify mirror))
-  )
-  (gr_text + (at 92.075 50.673) (layer B.SilkS)
-    (effects (font (size 1.5 1.5) (thickness 0.3)) (justify mirror))
-  )
-  (gr_text + (at 60.325 50.673) (layer B.SilkS)
-    (effects (font (size 1.5 1.5) (thickness 0.3)) (justify mirror))
-  )
-  (gr_text - (at 60.325 53.213) (layer B.SilkS)
-    (effects (font (size 1.5 1.5) (thickness 0.3)) (justify mirror))
-  )
   (gr_arc (start 55 45) (end 55 40) (angle -90) (layer Edge.Cuts) (width 0.15))
   (gr_arc (start 105 45) (end 110 45) (angle -90) (layer Edge.Cuts) (width 0.15))
@@
   (segment (start 72.7 155.4) (end 72.6 155.5) (width 0.3) (layer F.Cu) (net 3))
   (segment (start 63.9 160) (end 55 160) (width 0.3) (layer B.Cu) (net 3) (status 20))
-  (segment (start 78.25 135) (end 80 136.75) (width 0.3) (layer F.Cu) (net 3) (status 20))
-  (segment (start 69 135) (end 78.25 135) (width 0.3) (layer F.Cu) (net 3) (status 10))
-  (segment (start 89.25 136.75) (end 91 135) (width 0.3) (layer F.Cu) (net 3) (status 30))
-  (segment (start 80 136.75) (end 89.25 136.75) (width 0.3) (layer F.Cu) (net 3) (status 30))
   (segment (start 102.199999 42.199999) (end 105 45) (width 0.3) (layer F.Cu) (net 3) (status 20))
   (segment (start 61.618377 42.199999) (end 102.199999 42.199999) (width 0.3) (layer F.Cu) (net 3))
@@
   (segment (start 83.25 156.2) (end 84.192878 156.2) (width 0.3) (layer F.Cu) (net 3))
   (segment (start 85.492889 157.500011) (end 85.492889 158.567891) (width 0.3) (layer F.Cu) (net 3))
+  (via (at 70 135) (size 0.8) (drill 0.4) (layers F.Cu B.Cu) (net 3))
+  (segment (start 80 136.75) (end 71.75 136.75) (width 0.3) (layer F.Cu) (net 3))
+  (segment (start 71.75 136.75) (end 70 135) (width 0.3) (layer F.Cu) (net 3))
+  (segment (start 70 135) (end 69 135) (width 0.3) (layer B.Cu) (net 3))
   (via (at 83.474968 141.974957) (size 0.6) (drill 0.3) (layers F.Cu B.Cu) (net 4))
   (segment (start 83.899232 141.974957) (end 83.474968 141.974957) (width 0.15) (layer F.Cu) (net 4))
@@
   (segment (start 83.899967 139.477037) (end 83.577004 139.8) (width 0.15) (layer B.Cu) (net 19))
   (segment (start 83.899967 47.149967) (end 83.899967 139.477037) (width 0.15) (layer B.Cu) (net 19))
-  (via (at 72.7 139.20001) (size 0.6) (drill 0.3) (layers F.Cu B.Cu) (net 20))
-  (segment (start 74 141.5) (end 74 140.50001) (width 0.15) (layer F.Cu) (net 20) (status 10))
-  (segment (start 74 140.50001) (end 72.7 139.20001) (width 0.15) (layer F.Cu) (net 20))
-  (segment (start 72.400001 130.375723) (end 72.400001 138.900011) (width 0.15) (layer B.Cu) (net 20))
-  (segment (start 72.400001 138.900011) (end 72.7 139.20001) (width 0.15) (layer B.Cu) (net 20))
+  (via (at 72.600001 139.6) (size 0.6) (drill 0.3) (layers F.Cu B.Cu) (net 20))
+  (segment (start 74 140.9) (end 72.7 139.6) (width 0.15) (layer F.Cu) (net 20))
+  (segment (start 74 141.5) (end 74 140.9) (width 0.15) (layer F.Cu) (net 20))
+  (segment (start 72.7 139.6) (end 72.600001 139.6) (width 0.15) (layer F.Cu) (net 20))
+  (segment (start 71.2 138.199999) (end 72.600001 139.6) (width 0.15) (layer B.Cu) (net 20))
+  (segment (start 71.2 129.175722) (end 71.2 138.199999) (width 0.15) (layer B.Cu) (net 20))
   (segment (start 62.800011 105.625732) (end 62.800011 120.775733) (width 0.15) (layer B.Cu) (net 20))
-  (segment (start 60 83.25) (end 62.099967 85.349967) (width 0.15) (layer B.Cu) (net 20))
-  (segment (start 62.800011 120.775733) (end 72.400001 130.375723) (width 0.15) (layer B.Cu) (net 20))
   (segment (start 62.099967 104.925688) (end 62.800011 105.625732) (width 0.15) (layer B.Cu) (net 20))
   (segment (start 62.099967 85.349967) (end 62.099967 104.925688) (width 0.15) (layer B.Cu) (net 20))
-  (via (at 70.9 139.7) (size 0.6) (drill 0.3) (layers F.Cu B.Cu) (net 21))
-  (segment (start 70 140.6) (end 70.9 139.7) (width 0.15) (layer F.Cu) (net 21))
-  (segment (start 70 141.5) (end 70 140.6) (width 0.15) (layer F.Cu) (net 21) (status 10))
-  (segment (start 72.1 138.5) (end 70.9 139.7) (width 0.15) (layer B.Cu) (net 21))
-  (segment (start 72.1 130.5) (end 72.1 138.5) (width 0.15) (layer B.Cu) (net 21))
-  (segment (start 62.5 105.75) (end 62.5 120.9) (width 0.15) (layer B.Cu) (net 21))
+  (segment (start 62.800011 120.775733) (end 71.2 129.175722) (width 0.15) (layer B.Cu) (net 20))
+  (segment (start 60 83.25) (end 62.099967 85.349967) (width 0.15) (layer B.Cu) (net 20))
+  (segment (start 70.549988 139.999999) (end 70.849987 139.7) (width 0.15) (layer F.Cu) (net 21))
+  (segment (start 70 141.5) (end 70 140.549987) (width 0.15) (layer F.Cu) (net 21))
+  (segment (start 70 140.549987) (end 70.549988 139.999999) (width 0.15) (layer F.Cu) (net 21))
+  (via (at 70.849987 139.7) (size 0.6) (drill 0.3) (layers F.Cu B.Cu) (net 21))
+  (segment (start 70.849987 129.249988) (end 70.849987 139.275736) (width 0.15) (layer B.Cu) (net 21))
+  (segment (start 70.849987 139.275736) (end 70.849987 139.7) (width 0.15) (layer B.Cu) (net 21))
   (segment (start 60 103.25) (end 62.5 105.75) (width 0.15) (layer B.Cu) (net 21))
-  (segment (start 62.5 120.9) (end 72.1 130.5) (width 0.15) (layer B.Cu) (net 21))
+  (segment (start 62.5 105.75) (end 62.5 120.900001) (width 0.15) (layer B.Cu) (net 21))
+  (segment (start 62.5 120.900001) (end 70.849987 129.249988) (width 0.15) (layer B.Cu) (net 21))
   (via (at 79.300002 140) (size 0.6) (drill 0.3) (layers F.Cu B.Cu) (net 22))
   (segment (start 78.700002 140.6) (end 79.300002 140) (width 0.15) (layer F.Cu) (net 22))

Commit message: Added dimensions. Changed resistor value for LEDs. Fixed mode switch code
Parts:
- RN1, RN2, RN3: value 330 -> 1K
Changed lines of the file:
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@@
   (general
     (thickness 1.6)
-    (drawings 14)
+    (drawings 23)
     (tracks 618)
     (zones 0)
@@
   (layers
     (0 F.Cu signal)
-    (31 B.Cu signal)
-    (34 B.Paste user)
-    (35 F.Paste user)
-    (36 B.SilkS user)
+    (31 B.Cu signal hide)
+    (34 B.Paste user hide)
+    (35 F.Paste user hide)
+    (36 B.SilkS user hide)
     (37 F.SilkS user)
-    (38 B.Mask user)
-    (39 F.Mask user)
-    (44 Edge.Cuts user)
-    (45 Margin user)
-    (46 B.CrtYd user)
-    (47 F.CrtYd user)
+    (38 B.Mask user hide)
+    (39 F.Mask user hide)
+    (44 Edge.Cuts user hide)
+    (45 Margin user hide)
+    (46 B.CrtYd user hide)
+    (47 F.CrtYd user hide)
     (48 B.Fab user hide)
     (49 F.Fab user)
@@
       (effects (font (size 1 1) (thickness 0.15)))
     )
-    (fp_text value 330 (at 3 2.4625) (layer F.Fab)
+    (fp_text value 1K (at 3 2.4625) (layer F.Fab)
       (effects (font (size 1 1) (thickness 0.15)))
     )
@@
       (effects (font (size 1 1) (thickness 0.15)))
     )
-    (fp_text value 330 (at 3 2) (layer F.Fab)
+    (fp_text value 1K (at 3 2) (layer F.Fab)
       (effects (font (size 1 1) (thickness 0.15)))
     )
@@
       (effects (font (size 1 1) (thickness 0.15)))
     )
-    (fp_text value 330 (at 3 1.5375) (layer F.Fab)
+    (fp_text value 1K (at 3 1.5375) (layer F.Fab)
       (effects (font (size 1 1) (thickness 0.15)))
     )
@@
     )
   )
+  (dimension 25 (width 0.15) (layer F.Fab)
+    (gr_text "25.000 mm" (at 29.7 57.5 270) (layer F.Fab)
+      (effects (font (size 1 1) (thickness 0.15)))
+    )
+    (feature1 (pts (xy 60 70) (xy 30.413579 70)))
+    (feature2 (pts (xy 60 45) (xy 30.413579 45)))
+    (crossbar (pts (xy 31 45) (xy 31 70)))
+    (arrow1a (pts (xy 31 70) (xy 30.413579 68.873496)))
+    (arrow1b (pts (xy 31 70) (xy 31.586421 68.873496)))
+    (arrow2a (pts (xy 31 45) (xy 30.413579 46.126504)))
+    (arrow2b (pts (xy 31 45) (xy 31.586421 46.126504)))
+  )
+  (dimension 17.750018 (width 0.15) (layer F.Fab)
+    (gr_text "17.750 mm" (at 113.312825 151.104823 -89.91930177) (layer F.Fab)
+      (effects (font (size 1 1) (thickness 0.15)))
+    )
+    (feature1 (pts (xy 98.975 142.25) (xy 112.586746 142.230829)))
+    (feature2 (pts (xy 99 160) (xy 112.611746 159.980829)))
+    (crossbar (pts (xy 112.025326 159.981654) (xy 112.000326 142.231654)))
+    (arrow1a (pts (xy 112.000326 142.231654) (xy 112.588333 143.357331)))
+    (arrow1b (pts (xy 112.000326 142.231654) (xy 111.415492 143.358983)))
+    (arrow2a (pts (xy 112.025326 159.981654) (xy 112.61016 158.854325)))
+    (arrow2b (pts (xy 112.025326 159.981654) (xy 111.437319 158.855977)))
+  )
+  (dimension 25 (width 0.15) (layer F.Fab)
+    (gr_text "25.000 mm" (at 67.5 21.2) (layer F.Fab)
+      (effects (font (size 1 1) (thickness 0.15)))
+    )
+    (feature1 (pts (xy 55 40) (xy 55 21.913579)))
+    (feature2 (pts (xy 80 40) (xy 80 21.913579)))
+    (crossbar (pts (xy 80 22.5) (xy 55 22.5)))
+    (arrow1a (pts (xy 55 22.5) (xy 56.126504 21.913579)))
+    (arrow1b (pts (xy 55 22.5) (xy 56.126504 23.086421)))
+    (arrow2a (pts (xy 80 22.5) (xy 78.873496 21.913579)))
+    (arrow2b (pts (xy 80 22.5) (xy 78.873496 23.086421)))
+  )
+  (dimension 115 (width 0.15) (layer F.Fab)
+    (gr_text "115.000 mm" (at 116.235 102.5 270) (layer F.Fab)
+      (effects (font (size 1 1) (thickness 0.15)))
+    )
+    (feature1 (pts (xy 105 160) (xy 115.521421 160)))
+    (feature2 (pts (xy 105 45) (xy 115.521421 45)))
+    (crossbar (pts (xy 114.935 45) (xy 114.935 160)))
+    (arrow1a (pts (xy 114.935 160) (xy 114.348579 158.873496)))
+    (arrow1b (pts (xy 114.935 160) (xy 115.521421 158.873496)))
+    (arrow2a (pts (xy 114.935 45) (xy 114.348579 46.126504)))
+    (arrow2b (pts (xy 114.935 45) (xy 115.521421 46.126504)))
+  )
+  (dimension 50 (width 0.15) (layer F.Fab)
+    (gr_text "50.000 mm" (at 80 174.02) (layer F.Fab)
+      (effects (font (size 1 1) (thickness 0.15)))
+    )
+    (feature1 (pts (xy 105 160) (xy 105 173.306421)))
+    (feature2 (pts (xy 55 160) (xy 55 173.306421)))
+    (crossbar (pts (xy 55 172.72) (xy 105 172.72)))
+    (arrow1a (pts (xy 105 172.72) (xy 103.873496 173.306421)))
+    (arrow1b (pts (xy 105 172.72) (xy 103.873496 172.133579)))
+    (arrow2a (pts (xy 55 172.72) (xy 56.126504 173.306421)))
+    (arrow2b (pts (xy 55 172.72) (xy 56.126504 172.133579)))
+  )
+  (dimension 20 (width 0.15) (layer F.Fab)
+    (gr_text "20.000 mm" (at 70 26.005) (layer F.Fab)
+      (effects (font (size 1 1) (thickness 0.15)))
+    )
+    (feature1 (pts (xy 80 70) (xy 80 26.718579)))
+    (feature2 (pts (xy 60 70) (xy 60 26.718579)))
+    (crossbar (pts (xy 60 27.305) (xy 80 27.305)))
+    (arrow1a (pts (xy 80 27.305) (xy 78.873496 27.891421)))
+    (arrow1b (pts (xy 80 27.305) (xy 78.873496 26.718579)))
+    (arrow2a (pts (xy 60 27.305) (xy 61.126504 27.891421)))
+    (arrow2b (pts (xy 60 27.305) (xy 61.126504 26.718579)))
+  )
+  (dimension 37.95 (width 0.15) (layer F.Fab)
+    (gr_text "37.950 mm" (at 80 170.845) (layer F.Fab)
+      (effects (font (size 1 1) (thickness 0.15)))
+    )
+    (feature1 (pts (xy 98.975 142.25) (xy 98.975 170.131421)))
+    (feature2 (pts (xy 61.025 142.25) (xy 61.025 170.131421)))
+    (crossbar (pts (xy 61.025 169.545) (xy 98.975 169.545)))
+    (arrow1a (pts (xy 98.975 169.545) (xy 97.848496 170.131421)))
+    (arrow1b (pts (xy 98.975 169.545) (xy 97.848496 168.958579)))
+    (arrow2a (pts (xy 61.025 169.545) (xy 62.151504 170.131421)))
+    (arrow2b (pts (xy 61.025 169.545) (xy 62.151504 168.958579)))
+  )
+  (dimension 15 (width 0.15) (layer F.Fab)
+    (gr_text "15.000 mm" (at 30.45 134.75 270) (layer F.Fab)
+      (effects (font (size 1 1) (thickness 0.15)))
+    )
+    (feature1 (pts (xy 61.025 142.25) (xy 31.163579 142.25)))
+    (feature2 (pts (xy 61.025 127.25) (xy 31.163579 127.25)))
+    (crossbar (pts (xy 31.75 127.25) (xy 31.75 142.25)))
+    (arrow1a (pts (xy 31.75 142.25) (xy 31.163579 141.123496)))
+    (arrow1b (pts (xy 31.75 142.25) (xy 32.336421 141.123496)))
+    (arrow2a (pts (xy 31.75 127.25) (xy 31.163579 128.376504)))
+    (arrow2b (pts (xy 31.75 127.25) (xy 32.336421 128.376504)))
+  )
+  (dimension 20 (width 0.15) (layer F.Fab)
+    (gr_text "20.000 mm" (at 29.815 80 270) (layer F.Fab)
+      (effects (font (size 1 1) (thickness 0.15)))
+    )
+    (feature1 (pts (xy 60 90) (xy 30.528579 90)))
+    (feature2 (pts (xy 60 70) (xy 30.528579 70)))
+    (crossbar (pts (xy 31.115 70) (xy 31.115 90)))
+    (arrow1a (pts (xy 31.115 90) (xy 30.528579 88.873496)))
+    (arrow1b (pts (xy 31.115 90) (xy 31.701421 88.873496)))
+    (arrow2a (pts (xy 31.115 70) (xy 30.528579 71.126504)))
+    (arrow2b (pts (xy 31.115 70) (xy 31.701421 71.126504)))
+  )
   (gr_text JLCJLCJLCJLC (at 80 163.068) (layer B.SilkS)
