File: MerlinGame.sch (KiCad schematic (older format))
At the start: 39 parts, among them J1 AVR-ISP-6, J2 BATTERY, SW1 0, SW10 9, SW11 10, SW12 NEW GAME, SW13 SAME GAME, SW14 HIT ME, SW15 COMP TURN, SW16 POWER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

Commit message: Routing
Parts:
- RN1, RN2, RN3: value 1K -> 330
Other:
- moved on the sheet: J1
Changed lines of the file:
@@
 P 8200 1350
 F 0 "RN1" V 7750 1200 50  0000 C CNN
-F 1 "1K" V 7850 1200 50  0000 C CNN
+F 1 "330" V 7850 1200 50  0000 C CNN
 F 2 "Resistor_SMD:R_Array_Convex_4x1206" V 8475 1350 50  0001 C CNN
 F 3 "~" H 8200 1350 50  0001 C CNN
@@
 P 8200 1750
 F 0 "RN2" V 7350 1800 50  0000 C CNN
-F 1 "1K" V 7450 1800 50  0000 C CNN
+F 1 "330" V 7450 1800 50  0000 C CNN
 F 2 "Resistor_SMD:R_Array_Convex_4x1206" V 8475 1750 50  0001 C CNN
 F 3 "~" H 8200 1750 50  0001 C CNN
@@
 P 8200 2150
 F 0 "RN3" V 6950 2400 50  0000 C CNN
-F 1 "1K" V 7050 2400 50  0000 C CNN
+F 1 "330" V 7050 2400 50  0000 C CNN
 F 2 "Resistor_SMD:R_Array_Convex_4x1206" V 8475 2150 50  0001 C CNN
 F 3 "~" H 8200 2150 50  0001 C CNN
@@
 	4600 700  2550 700
 Connection ~ 4600 700
-$Comp
-L Connector:AVR-ISP-6 J1
-U 1 1 5DA20642
-P 1700 6800
-F 0 "J1" H 1420 6896 50  0000 R CNN
-F 1 "AVR-ISP-6" H 1420 6805 50  0000 R CNN
-F 2 "Connector:Tag-Connect_TC2030-IDC-NL_2x03_P1.27mm_Vertical" V 1450 6850 50  0001 C CNN
-F 3 " ~" H 425 6250 50  0001 C CNN
-	1    1700 6800
-	1    0    0    -1
-$EndComp
 Text GLabel 9250 4800 2    50   Input ~ 0
 ~RESET
@@
 	1    0    0    -1
 $EndComp
-Text GLabel 2250 6700 2    50   Output ~ 0
+Text GLabel 2000 6700 2    50   Output ~ 0
 MOSI
-Text GLabel 2250 6600 2    50   Input ~ 0
+Text GLabel 2000 6600 2    50   Input ~ 0
 MISO
-Text GLabel 2250 6800 2    50   Output ~ 0
+Text GLabel 2000 6800 2    50   Output ~ 0
 SCK
-Text GLabel 2250 6900 2    50   Output ~ 0
+Text GLabel 2000 6900 2    50   Output ~ 0
 ~RESET
 Wire Wire Line
-	2100 6600 2250 6600
-Wire Wire Line
-	2100 6700 2250 6700
-Wire Wire Line
-	2100 6800 2250 6800
-Wire Wire Line
-	2100 6900 2250 6900
+	1850 6600 2000 6600
+Wire Wire Line
+	1850 6700 2000 6700
+Wire Wire Line
+	1850 6800 2000 6800
+Wire Wire Line
+	1850 6900 2000 6900
 $Comp
 L power:GND #PWR0106
 U 1 1 5DA44CAC
-P 1600 7300
-F 0 "#PWR0106" H 1600 7050 50  0001 C CNN
-F 1 "GND" H 1605 7127 50  0000 C CNN
-F 2 "" H 1600 7300 50  0001 C CNN
-F 3 "" H 1600 7300 50  0001 C CNN
-	1    1600 7300
+P 1350 7300
+F 0 "#PWR0106" H 1350 7050 50  0001 C CNN
+F 1 "GND" H 1355 7127 50  0000 C CNN
+F 2 "" H 1350 7300 50  0001 C CNN
+F 3 "" H 1350 7300 50  0001 C CNN
+	1    1350 7300
 	1    0    0    -1
 $EndComp
@@
 L power:VCC #PWR0107
 U 1 1 5DA44DCE
-P 1600 6250
-F 0 "#PWR0107" H 1600 6100 50  0001 C CNN
-F 1 "VCC" H 1617 6423 50  0000 C CNN
-F 2 "" H 1600 6250 50  0001 C CNN
-F 3 "" H 1600 6250 50  0001 C CNN
-	1    1600 6250
+P 1350 6250
+F 0 "#PWR0107" H 1350 6100 50  0001 C CNN
+F 1 "VCC" H 1367 6423 50  0000 C CNN
+F 2 "" H 1350 6250 50  0001 C CNN
+F 3 "" H 1350 6250 50  0001 C CNN
+	1    1350 6250
 	1    0    0    -1
 $EndComp
@@
 	1900 5200 2050 5200
 Wire Wire Line
-	1600 7200 1600 7300
-Wire Wire Line
-	1600 6250 1600 6300
+	1350 7200 1350 7300
+Wire Wire Line
+	1350 6250 1350 6300
 Wire Wire Line
 	7700 6050 7700 6000
@@
 Wire Wire Line
 	6500 3800 6500 3750
-Wire Bus Line
-	6250 4850 6250 5550
-Wire Bus Line
-	4850 4850 4850 5550
-Wire Bus Line
-	5200 5300 5200 6000
-Wire Bus Line
-	6400 700  6400 3050
-Wire Bus Line
-	2550 700  2550 3050
-Wire Bus Line
-	3800 4350 3800 6000
-Wire Bus Line
-	850  1950 850  4350
-Wire Bus Line
-	4800 1950 4800 4350
-Wire Bus Line
-	2100 850  2100 2950
-Wire Bus Line
-	4100 850  4100 3550
-Wire Bus Line
-	4600 700  4600 3650
-Wire Bus Line
-	8850 5100 8850 6350
-Wire Bus Line
-	8750 5500 8750 6450
-Wire Bus Line
-	2800 1350 2800 4350
-Wire Bus Line
-	6000 850  6000 4850
-Wire Bus Line
-	7600 700  7600 2050
-Wire Bus Line
-	8750 700  8750 4500
 Text Label 6850 3600 0    50   ~ 0
 ADC7
 Text Label 6900 3300 0    50   ~ 0
 AREF
+$Comp
+L Connector:AVR-ISP-6 J1
+U 1 1 5DA20642
+P 1450 6800
+F 0 "J1" H 1170 6896 50  0000 R CNN
+F 1 "AVR-ISP-6" H 1170 6805 50  0000 R CNN
+F 2 "Connector:Tag-Connect_TC2030-IDC-NL_2x03_P1.27mm_Vertical" V 1200 6850 50  0001 C CNN
+F 3 " ~" H 175 6250 50  0001 C CNN
+	1    1450 6800
+	1    0    0    -1
+$EndComp
+Wire Bus Line
+	5200 5300 5200 6000
+Wire Bus Line
+	4850 4850 4850 5550
+Wire Bus Line
+	6250 4850 6250 5550
+Wire Bus Line
+	6400 700  6400 3050
+Wire Bus Line
+	2550 700  2550 3050
+Wire Bus Line
+	3800 4350 3800 6000
+Wire Bus Line
+	850  1950 850  4350
+Wire Bus Line
+	4800 1950 4800 4350
+Wire Bus Line
+	2100 850  2100 2950
+Wire Bus Line
+	6000 850  6000 4850
+Wire Bus Line
+	4100 850  4100 3550
+Wire Bus Line
+	2800 1350 2800 4350
+Wire Bus Line
+	8750 5500 8750 6450
+Wire Bus Line
+	8850 5100 8850 6350
+Wire Bus Line
+	4600 700  4600 3650
+Wire Bus Line
+	7600 700  7600 2050
+Wire Bus Line
+	8750 700  8750 4500
 $EndSCHEMATC

Commit message: Updated silkscreen, added plots
Parts:
- C1, C2: value 22pF -> 18pF
Changed lines of the file:
@@
 P 10050 3850
 F 0 "C1" V 9821 3850 50  0000 C CNN
-F 1 "22pF" V 9912 3850 50  0000 C CNN
+F 1 "18pF" V 9912 3850 50  0000 C CNN
 F 2 "Capacitor_SMD:C_0805_2012Metric_Pad1.15x1.40mm_HandSolder" H 10050 3850 50  0001 C CNN
 F 3 "~" H 10050 3850 50  0001 C CNN
@@
 P 10050 4050
 F 0 "C2" V 9800 4050 50  0000 C CNN
-F 1 "22pF" V 9900 4050 50  0000 C CNN
+F 1 "18pF" V 9900 4050 50  0000 C CNN
 F 2 "Capacitor_SMD:C_0805_2012Metric_Pad1.15x1.40mm_HandSolder" H 10050 4050 50  0001 C CNN
 F 3 "~" H 10050 4050 50  0001 C CNN

Commit message: Removed battery holes
Parts:
- removed MH5: BATTERY1, MountingHole:MountingHole_2.7mm_Pad, symbol Mechanical:MountingHole_Pad
- removed MH6: BATTERY2, MountingHole:MountingHole_2.7mm_Pad, symbol Mechanical:MountingHole_Pad
Other:
- moved on the sheet: MH1, MH2, MH3, MH4
Changed lines of the file:
@@
-$EndComp
-$Comp
-L Mechanical:MountingHole_Pad MH6
-U 1 1 5DA4CD65
-P 5700 7600
-F 0 "MH6" H 5800 7651 50  0000 L CNN
-F 1 "BATTERY2" H 5800 7560 50  0000 L CNN
-F 2 "MountingHole:MountingHole_2.7mm_Pad" H 5700 7600 50  0001 C CNN
-F 3 "~" H 5700 7600 50  0001 C CNN
-	1    5700 7600
-	1    0    0    -1
-$EndComp
-$Comp
-L Mechanical:MountingHole_Pad MH5
-U 1 1 5DA4CDC1
-P 5200 7600
-F 0 "MH5" H 5300 7651 50  0000 L CNN
-F 1 "BATTERY1" H 5300 7560 50  0000 L CNN
-F 2 "MountingHole:MountingHole_2.7mm_Pad" H 5200 7600 50  0001 C CNN
-F 3 "~" H 5200 7600 50  0001 C CNN
-	1    5200 7600
-	1    0    0    -1
 $EndComp
 $Comp
 L Mechanical:MountingHole_Pad MH2
 U 1 1 5DA4CF95
-P 4000 7600
-F 0 "MH2" H 4100 7651 50  0000 L CNN
-F 1 "CASE" H 4100 7560 50  0000 L CNN
-F 2 "MountingHole:MountingHole_2.7mm_Pad" H 4000 7600 50  0001 C CNN
-F 3 "~" H 4000 7600 50  0001 C CNN
-	1    4000 7600
+P 4100 6850
+F 0 "MH2" H 4200 6901 50  0000 L CNN
+F 1 "CASE" H 4200 6810 50  0000 L CNN
+F 2 "MountingHole:MountingHole_2.7mm_Pad" H 4100 6850 50  0001 C CNN
+F 3 "~" H 4100 6850 50  0001 C CNN
+	1    4100 6850
 	1    0    0    -1
 $EndComp
@@
 L Mechanical:MountingHole_Pad MH1
 U 1 1 5DA4CF9B
-P 3600 7600
-F 0 "MH1" H 3700 7651 50  0000 L CNN
-F 1 "CASE" H 3700 7560 50  0000 L CNN
-F 2 "MountingHole:MountingHole_2.7mm_Pad" H 3600 7600 50  0001 C CNN
-F 3 "~" H 3600 7600 50  0001 C CNN
-	1    3600 7600
+P 3700 6850
+F 0 "MH1" H 3800 6901 50  0000 L CNN
+F 1 "CASE" H 3800 6810 50  0000 L CNN
+F 2 "MountingHole:MountingHole_2.7mm_Pad" H 3700 6850 50  0001 C CNN
+F 3 "~" H 3700 6850 50  0001 C CNN
+	1    3700 6850
 	1    0    0    -1
 $EndComp
@@
 L Mechanical:MountingHole_Pad MH4
 U 1 1 5DA50A12
-P 4800 7600
-F 0 "MH4" H 4900 7646 50  0000 L CNN
-F 1 "CASE" H 4900 7555 50  0000 L CNN
-F 2 "MountingHole:MountingHole_2.7mm_Pad" H 4800 7600 50  0001 C CNN
-F 3 "~" H 4800 7600 50  0001 C CNN
-	1    4800 7600
+P 4900 6850
+F 0 "MH4" H 5000 6896 50  0000 L CNN
+F 1 "CASE" H 5000 6805 50  0000 L CNN
+F 2 "MountingHole:MountingHole_2.7mm_Pad" H 4900 6850 50  0001 C CNN
+F 3 "~" H 4900 6850 50  0001 C CNN
+	1    4900 6850
 	1    0    0    -1
 $EndComp
@@
 L Mechanical:MountingHole_Pad MH3
 U 1 1 5DA50A18
-P 4400 7600
-F 0 "MH3" H 4500 7646 50  0000 L CNN
-F 1 "CASE" H 4500 7555 50  0000 L CNN
-F 2 "MountingHole:MountingHole_2.7mm_Pad" H 4400 7600 50  0001 C CNN
-F 3 "~" H 4400 7600 50  0001 C CNN
-	1    4400 7600
+P 4500 6850
+F 0 "MH3" H 4600 6896 50  0000 L CNN
+F 1 "CASE" H 4600 6805 50  0000 L CNN
+F 2 "MountingHole:MountingHole_2.7mm_Pad" H 4500 6850 50  0001 C CNN
+F 3 "~" H 4500 6850 50  0001 C CNN
+	1    4500 6850
 	1    0    0    -1
 $EndComp
@@
 L power:GND #PWR0108
 U 1 1 5DA5C72D
-P 5700 7800
-F 0 "#PWR0108" H 5700 7550 50  0001 C CNN
-F 1 "GND" H 5705 7627 50  0000 C CNN
-F 2 "" H 5700 7800 50  0001 C CNN
-F 3 "" H 5700 7800 50  0001 C CNN
-	1    5700 7800
-	1    0    0    -1
-$EndComp
-Wire Wire Line
-	3600 7700 4000 7700
-Wire Wire Line
-	5700 7700 5700 7800
-Connection ~ 5700 7700
-Connection ~ 4000 7700
-Wire Wire Line
-	4000 7700 4400 7700
-Connection ~ 4400 7700
-Wire Wire Line
-	4400 7700 4800 7700
-Connection ~ 4800 7700
-Wire Wire Line
-	4800 7700 5200 7700
-Connection ~ 5200 7700
-Wire Wire Line
-	5200 7700 5700 7700
+P 4350 7050
+F 0 "#PWR0108" H 4350 6800 50  0001 C CNN
+F 1 "GND" H 4355 6877 50  0000 C CNN
+F 2 "" H 4350 7050 50  0001 C CNN
+F 3 "" H 4350 7050 50  0001 C CNN
+	1    4350 7050
+	1    0    0    -1
+$EndComp
+Wire Wire Line
+	3700 6950 4100 6950
+Wire Wire Line
+	4350 6950 4350 7050
+Connection ~ 4100 6950
+Wire Wire Line
+	4100 6950 4350 6950
+Connection ~ 4500 6950
+Wire Wire Line
+	4500 6950 4900 6950
 Entry Wire Line
 	6150 5200 6250 5100
@@
 	1    0    0    -1
 $EndComp
+Connection ~ 4350 6950
+Wire Wire Line
+	4350 6950 4500 6950
 Wire Bus Line
 	5200 5300 5200 6000

Commit message: Added dimensions. Changed resistor value for LEDs. Fixed mode switch code
Parts:
- RN1, RN2, RN3: value 330 -> 1K
Changed lines of the file:
@@
 P 8200 1350
 F 0 "RN1" V 7750 1200 50  0000 C CNN
-F 1 "330" V 7850 1200 50  0000 C CNN
+F 1 "1K" V 7850 1200 50  0000 C CNN
 F 2 "Resistor_SMD:R_Array_Convex_4x1206" V 8475 1350 50  0001 C CNN
 F 3 "~" H 8200 1350 50  0001 C CNN
@@
 P 8200 1750
 F 0 "RN2" V 7350 1800 50  0000 C CNN
-F 1 "330" V 7450 1800 50  0000 C CNN
+F 1 "1K" V 7450 1800 50  0000 C CNN
 F 2 "Resistor_SMD:R_Array_Convex_4x1206" V 8475 1750 50  0001 C CNN
 F 3 "~" H 8200 1750 50  0001 C CNN
@@
 P 8200 2150
 F 0 "RN3" V 6950 2400 50  0000 C CNN
-F 1 "330" V 7050 2400 50  0000 C CNN
+F 1 "1K" V 7050 2400 50  0000 C CNN
 F 2 "Resistor_SMD:R_Array_Convex_4x1206" V 8475 2150 50  0001 C CNN
 F 3 "~" H 8200 2150 50  0001 C CNN
