File: WizardGame.sch (KiCad schematic (older format))
At the start: 37 parts, among them J1 AVR-ISP-6, J2 BATTERY, SW1 0, SW10 9, SW11 10, SW12 NEW GAME, SW13 SAME GAME, SW14 HIT ME, SW15 COMP TURN, SW16 POWER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

Commit message: Renamed, cleanup
Parts:
- U1: symbol MerlinGame-rescue:ATmega328P-AU-MCU_Microchip_ATmega -> MCU_Microchip_ATmega:ATmega328P-AU
Changed lines of the file:
@@
 EESchema Schematic File Version 4
-LIBS:MerlinGame-cache
 EELAYER 30 0
 EELAYER END
@@
 encoding utf-8
 Sheet 1 1
-Title "Merlin"
+Title "Wizard Electronic Game"
 Date "2019-10-10"
 Rev "A"
@@
 $EndComp
 $Comp
-L MerlinGame-rescue:ATmega328P-AU-MCU_Microchip_ATmega U1
+L MCU_Microchip_ATmega:ATmega328P-AU U1
 U 1 1 5D8A88CB
 P 7700 4500
